File: pcb/phase.kicad_sch (KiCad schematic)
At the start: 9 parts, among them Q1 AON7544, Q2 AON7544

Commit message: Fix filenames
Parts:
- renumbered C1 to C2, NT1 to NT2, Q1 to Q3, Q2 to Q4, R5 to R10, R3 to R6, R2 to R7, R1 to R8, R4 to R9
Other:
- moved on the sheet: C2, NT2, Q3, Q4, R10, R6, R7, R8, R9

Commit message: Save
Parts:
- removed Q3, Q4: AON7544, User_Footprints:DFN3x3A_8L_EP1_P, symbol User_Symbols:AON7544
- added Q1, Q8: IAUCN08S7N013, symbol User_Symbols:NMOS_PWR
- C2: value 220n -> 470n
- R10: value R -> 33k
- R9: value 10k -> 1k
Connections:
- net PH: now also Q1.5 (D), Q1.6 (D), Q1.7 (D), Q1.8 (D), Q8.1 (S), Q8.2 (S), Q8.3 (S)
- net at R6.2: now also Q8.4 (G)
- net at R7.2: now also Q1.4 (G)
- net at R8.1, R9.1: now also Q1.1 (S), Q1.2 (S), Q1.3 (S)
- net GND renamed GNDPWR
- new net VDD: Q8.5 (D), Q8.6 (D), Q8.7 (D), Q8.8 (D)
Other:
- note added: "Max Regen 100A"
- moved on the sheet: C2, NT2, R10, R9

Commit message: Save
Parts:
- C2: footprint (none) -> Capacitor_SMD:C_0603_1608Metric
- R10: value 33k -> 3k3
- R9: value 1k -> 100R
- renumbered Q8 to Q2
Other:
- note added: "NTMFS6H801NLT1G 1.3mΩ -> 2.2mΩ 116nC -> 44nC"

Commit message: Save
Parts:
- added R26: 100R, Resistor_SMD:R_0402_1005Metric, symbol Device:R
- C11: renamed from C2; LCSC (none) -> C1623
- NT3: renamed from NT2; footprint (none) -> NetTie:NetTie-2_SMD_Pad0.5mm
- Q1: renamed from Q2; value IAUCN08S7N013 -> NTMFS6H801NLT1G; footprint (none) -> Package_SO:PowerPAK_SO-8_Single; LCSC (none) -> C900316
- Q2: renamed from Q1; value IAUCN08S7N013 -> NTMFS6H801NLT1G; footprint (none) -> Package_SO:PowerPAK_SO-8_Single; LCSC (none) -> C900316
- R10: renamed from R7; footprint (none) -> Resistor_SMD:R_0402_1005Metric; LCSC (none) -> C25077
- R11: renamed from R8; footprint (none) -> Resistor_SMD:R_2512_6332Metric; LCSC (none) -> C5375452
- R12: renamed from R9; footprint (none) -> Resistor_SMD:R_0402_1005Metric
- R13: renamed from R10; footprint (none) -> Resistor_SMD:R_0402_1005Metric; LCSC (none) -> C25890
- R9: renamed from R6; footprint (none) -> Resistor_SMD:R_0402_1005Metric; LCSC (none) -> C25077
Connections:
- net SNSL: now also R26.2; no longer NT3.2
- new net: NT3.2, R26.1
Other:
- note added: "IAUCN08S7N013 NTMFS6H801NLT1G 1.3mΩ -> 2.2mΩ 116nC -> 44nC"
- note removed: "NTMFS6H801NLT1G 1.3mΩ -> 2.2mΩ 116nC -> 44nC"
