File: pcb/small-foc.kicad_pcb (KiCad board)
At the start: 4 copper layers, 0 parts

Commit message: Save
Parts:
- added C11: 470n, Capacitor_SMD:C_0603_1608Metric, F.Cu at (65.6, 77.0)
- added C12: 470n, Capacitor_SMD:C_0603_1608Metric, F.Cu at (61.3, 93.4)
- added C13: 470n, Capacitor_SMD:C_0603_1608Metric, F.Cu at (65.6, 82.6)
- added C14: 12p, Capacitor_SMD:C_0402_1005Metric, F.Cu at (89.2, 82.8)
- added C15: 100n, Capacitor_SMD:C_0402_1005Metric, F.Cu at (87.2, 82.8)
- added C16: 12p, Capacitor_SMD:C_0402_1005Metric, F.Cu at (85.2, 82.8)
- added C17: 100n, Capacitor_SMD:C_0402_1005Metric, F.Cu at (83.2, 82.8)
- added C5: 100n, Capacitor_SMD:C_0402_1005Metric, F.Cu at (91.1, 82.8)
- added J1: Conn_ARM_SWD_TagConnect_TC2030-NL, Connector:Tag-Connect_TC2030-IDC-NL_2x03_P1.27mm_Vertical, F.Cu at (78.3, 74.0)
- added JP1: SolderJumper_2_Open, Jumper:SolderJumper-2_P1.3mm_Open_RoundedPad1.0x1.5mm, F.Cu at (90.3, 86.4)
- added NT2: NetTie_2, NetTie:NetTie-2_SMD_Pad0.5mm, F.Cu at (85.8, 85.4)
- added NT3: NetTie_2, NetTie:NetTie-2_SMD_Pad0.5mm, F.Cu at (68.0, 77.0)
- added NT4: NetTie_2, NetTie:NetTie-2_SMD_Pad0.5mm, F.Cu at (63.7, 93.4)
- added NT5: NetTie_2, NetTie:NetTie-2_SMD_Pad0.5mm, F.Cu at (68.0, 82.6)
- added Q1: NTMFS6H801NLT1G, Package_SO:PowerPAK_SO-8_Single, B.Cu at (124.3, 43.5)
- added Q2: NTMFS6H801NLT1G, Package_SO:PowerPAK_SO-8_Single, F.Cu at (124.3, 43.5)
- added Q3: NTMFS6H801NLT1G, Package_SO:PowerPAK_SO-8_Single, B.Cu at (124.3, 54.9)
- added Q4: NTMFS6H801NLT1G, Package_SO:PowerPAK_SO-8_Single, F.Cu at (124.3, 54.9)
- added Q5: NTMFS6H801NLT1G, Package_SO:PowerPAK_SO-8_Single, B.Cu at (124.3, 49.2)
- added Q6: NTMFS6H801NLT1G, Package_SO:PowerPAK_SO-8_Single, F.Cu at (124.3, 49.2)
- added R10: 10R, Resistor_SMD:R_0402_1005Metric, F.Cu at (73.9, 94.4)
- added R11: 1m, Resistor_SMD:R_2512_6332Metric, F.Cu at (116.8, 43.6)
- added R12: 100R, Resistor_SMD:R_0402_1005Metric, F.Cu at (71.6, 77.1)
- added R13: 3k3, Resistor_SMD:R_0402_1005Metric, F.Cu at (69.6, 76.8)
- added R14: 10R, Resistor_SMD:R_0402_1005Metric, F.Cu at (71.2, 88.8)
- added R15: 10R, Resistor_SMD:R_0402_1005Metric, F.Cu at (73.5, 88.8)
- added R16: 1m, Resistor_SMD:R_2512_6332Metric, F.Cu at (116.8, 54.8)
- added R17: 100R, Resistor_SMD:R_0402_1005Metric, F.Cu at (67.3, 93.5)
- added R18: 3k3, Resistor_SMD:R_0402_1005Metric, F.Cu at (65.4, 93.0)
- added R19: 10R, Resistor_SMD:R_0402_1005Metric, F.Cu at (71.7, 100.0)
- added R20: 10R, Resistor_SMD:R_0402_1005Metric, F.Cu at (73.9, 100.0)
- added R21: 1m, Resistor_SMD:R_2512_6332Metric, F.Cu at (116.8, 49.2)
- added R22: 100R, Resistor_SMD:R_0402_1005Metric, F.Cu at (71.6, 82.7)
- added R23: 3k3, Resistor_SMD:R_0402_1005Metric, F.Cu at (69.6, 82.6)
- added R24: 1k, Resistor_SMD:R_0402_1005Metric, F.Cu at (87.6, 85.6)
- added R25: 120, Resistor_SMD:R_1206_3216Metric, F.Cu at (74.5, 80.9)
- added R9: 10R, Resistor_SMD:R_0402_1005Metric, F.Cu at (71.7, 94.4)
- added REF**: MountingHole_3.5mm, MountingHole:MountingHole_3.5mm, F.Cu at (131.6, 43.4)
- added REF**: C_Elec_6.3x7.7, Capacitor_SMD:C_Elec_6.3x7.7, F.Cu at (106.8, 71.8)
- added REF**: C_Elec_6.3x7.7, Capacitor_SMD:C_Elec_6.3x7.7, F.Cu at (115.8, 71.8)
- added REF**: C_1210_3225Metric, Capacitor_SMD:C_1210_3225Metric, F.Cu at (107.6, 49.5)
- added REF**: C_1210_3225Metric, Capacitor_SMD:C_1210_3225Metric, F.Cu at (107.6, 55.9)
- added REF**: C_1210_3225Metric, Capacitor_SMD:C_1210_3225Metric, F.Cu at (107.6, 43.1)
- added REF**: C_1210_3225Metric, Capacitor_SMD:C_1210_3225Metric, F.Cu at (107.6, 46.3)
- added REF**: PinHeader_1x04_P1.00mm_Vertical, Connector_PinHeader_1.00mm:PinHeader_1x04_P1.00mm_Vertical, F.Cu at (113.8, 57.6)
- added REF**: MountingHole_3.5mm, MountingHole:MountingHole_3.5mm, F.Cu at (131.6, 54.8)
- added REF**: C_Elec_6.3x7.7, Capacitor_SMD:C_Elec_6.3x7.7, F.Cu at (115.8, 79.0)
- added REF**: C_0603_1608Metric, Capacitor_SMD:C_0603_1608Metric, B.Cu at (115.8, 42.8)
- added REF**: PinHeader_1x04_P1.00mm_Vertical, Connector_PinHeader_1.00mm:PinHeader_1x04_P1.00mm_Vertical, F.Cu at (113.7, 46.4)
- added REF**: C_0603_1608Metric, Capacitor_SMD:C_0603_1608Metric, B.Cu at (115.8, 52.8)
- added REF**: C_Elec_6.3x7.7, Capacitor_SMD:C_Elec_6.3x7.7, B.Cu at (123.8, 75.8)
- added REF**: C_1210_3225Metric, Capacitor_SMD:C_1210_3225Metric, B.Cu at (109.6, 52.7)
- added REF**: C_0603_1608Metric, Capacitor_SMD:C_0603_1608Metric, B.Cu at (115.8, 55.6)
- added REF**: C_0603_1608Metric, Capacitor_SMD:C_0603_1608Metric, B.Cu at (115.8, 47.1)
- added REF**: C_0603_1608Metric, Capacitor_SMD:C_0603_1608Metric, B.Cu at (115.8, 41.4)
- added REF**: C_0603_1608Metric, Capacitor_SMD:C_0603_1608Metric, B.Cu at (115.8, 44.2)
- added REF**: C_Elec_6.3x7.7, Capacitor_SMD:C_Elec_6.3x7.7, B.Cu at (106.8, 71.8)
- added REF**: C_1210_3225Metric, Capacitor_SMD:C_1210_3225Metric, B.Cu at (109.6, 49.5)
- added REF**: C_Elec_6.3x7.7, Capacitor_SMD:C_Elec_6.3x7.7, B.Cu at (106.8, 79.0)
- added REF**: C_Elec_6.3x7.7, Capacitor_SMD:C_Elec_6.3x7.7, F.Cu at (106.8, 79.0)
- added REF**: C_1210_3225Metric, Capacitor_SMD:C_1210_3225Metric, B.Cu at (109.6, 43.1)
- added REF**: C_0603_1608Metric, Capacitor_SMD:C_0603_1608Metric, B.Cu at (115.8, 51.3)
- added REF**: C_0603_1608Metric, Capacitor_SMD:C_0603_1608Metric, B.Cu at (115.8, 54.2)
- added REF**: C_1210_3225Metric, Capacitor_SMD:C_1210_3225Metric, B.Cu at (109.6, 46.3)
- added REF**: C_1210_3225Metric, Capacitor_SMD:C_1210_3225Metric, B.Cu at (109.6, 55.9)
- added REF**: C_0603_1608Metric, Capacitor_SMD:C_0603_1608Metric, B.Cu at (115.8, 49.9)
- added REF**: C_0603_1608Metric, Capacitor_SMD:C_0603_1608Metric, B.Cu at (115.8, 57.0)
- added REF**: C_0603_1608Metric, Capacitor_SMD:C_0603_1608Metric, B.Cu at (115.8, 45.6)
- added REF**: C_Elec_6.3x7.7, Capacitor_SMD:C_Elec_6.3x7.7, B.Cu at (115.8, 79.0)
- added REF**: C_Elec_6.3x7.7, Capacitor_SMD:C_Elec_6.3x7.7, B.Cu at (115.8, 71.8)
- added REF**: PinHeader_1x04_P1.00mm_Vertical, Connector_PinHeader_1.00mm:PinHeader_1x04_P1.00mm_Vertical, F.Cu at (113.7, 52.0)
- added REF**: C_0603_1608Metric, Capacitor_SMD:C_0603_1608Metric, B.Cu at (115.8, 48.5)
- added REF**: MountingHole_3.5mm, MountingHole:MountingHole_3.5mm, F.Cu at (131.6, 49.1)
- added REF**: C_1210_3225Metric, Capacitor_SMD:C_1210_3225Metric, F.Cu at (107.6, 52.7)
- added REF**: C_Elec_6.3x7.7, Capacitor_SMD:C_Elec_6.3x7.7, F.Cu at (123.8, 75.8)
- added REF**: MountingHole_3.5mm, MountingHole:MountingHole_3.5mm, F.Cu at (97.4, 54.8)
- added REF**: MountingHole_3.5mm, MountingHole:MountingHole_3.5mm, F.Cu at (97.4, 43.4)
- added U1: STSPIN32G4, Package_DFN_QFN:Texas_RGC0064B_VQFN-64-1EP_9x9mm_P0.5mm_EP4.25x4.25mm, F.Cu at (86.5, 75.7)
- added U2: TJA1044GTK/3, Package_SON:HVSON-8-1EP_3x3mm_P0.65mm_EP1.6x2.4mm, F.Cu at (78.5, 81.1)
- added Y1: 16MHz, Crystal:Crystal_SMD_3225-4Pin_3.2x2.5mm, F.Cu at (78.6, 86.4)

Commit message: Save
Parts:
- moved NT4 19.8 mm to (70.4, 74.8)
- moved C12 19.8 mm to (68.0, 74.8)
- moved R17 19.8 mm to (74.0, 74.9)
- moved R18 19.8 mm to (72.1, 74.4)
- moved R19 13.6 mm to (74.2, 86.6)
- moved R20 13.6 mm to (76.4, 86.6)
- moved NT5 12.0 mm to (70.4, 70.8)
- moved R23 12.0 mm to (72.0, 70.8)
- moved C13 12.0 mm to (68.0, 70.8)
- moved R22 12.0 mm to (74.0, 70.9)
- moved R10 10.3 mm to (76.9, 84.6)
- moved R9 10.3 mm to (74.7, 84.6)
- moved C11 10.2 mm to (67.8, 67.0)
- moved R12 10.2 mm to (73.8, 67.1)
- moved R13 10.2 mm to (71.8, 66.8)
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