File: pcb/small-foc.kicad_sch (KiCad schematic)
At the start: 17 parts, among them J1 Conn_ARM_SWD_TagConnect_TC203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, U1 STSPING4

Commit message: Save
Parts:
- removed U1: STSPING4, Package_DFN_QFN:Texas_RGC0064B_VQFN-64-1EP_9x9mm_P0.5mm_EP4.25x4.25mm, symbol User_Symbols:STSPING4
- added U1: STSPIN32G4, Package_DFN_QFN:Texas_RGC0064B_VQFN-64-1EP_9x9mm_P0.5mm_EP4.25x4.25mm, symbol User_Symbols:STSPIN32G4
Connections:
- net +3V3A: now also U1.26 (VREF+), U1.27 (VDDA)
- net BSTA: now also U1.41 (BOOT1)
- net BSTB: now also U1.38 (BOOT2)
- net BSTC: now also U1.35 (BOOT3)
- net GND: now also U1.59 (PB8), U1.65 (EPAD)
- net GNDPWR: now also U1.32 (PGND)
- net INHA: now also U1.43 (GHS1)
- net INHB: now also U1.40 (GHS2)
- net INHC: now also U1.37 (GHS3)
- net INLA: now also U1.29 (GLS1)
- net INLB: now also U1.30 (GLS2)
- net INLC: now also U1.31 (GLS3)
- net NRST: now also U1.8 (PG10)
- net PHA: now also U1.42 (OUT1)
- net PHB: now also U1.39 (OUT2)
- net PHC: now also U1.36 (OUT3)
- net SCREF: now also U1.52 (SCREF)
- net SWCLK: now also U1.50 (PA14)
- net SWDIO: now also U1.49 (PA13)
- net XTALI: now also U1.6 (PF0)
- net XTALO: now also U1.7 (PF1)
- new net: U1.1 (REG3/VDD), U1.2 (VBAT)
Other:
- moved on the sheet: J1

Commit message: Save
Parts:
- added R23, R24: 51k, symbol Device:R
- C10: value C -> 1n
- C9: value C -> 470n
- R18, R20: value R -> 33k
- R19, R21: value R -> 3k3
Connections:
- net SNSHA: now also U1.14 (PA1)
- net SNSHB: now also U1.20 (PA7)
- net SNSHC: now also U1.23 (PB0)
- net SNSLA: now also U1.16 (PA3)
- net SNSLB: now also U1.18 (PA5)
- net SNSLC: now also U1.25 (PB2)
- net VDD: now also R23.1, R24.1; no longer R18.1, R20.1
- new net: R20.1, R23.2
- new net: R18.1, R24.2
Other:
- note added: "75V VDD Max"
- note added: "Gate driver GND"
- note added: "T = 300khz"
- note added: "T = 600hz"
- moved on the sheet: C9

Commit message: Save
Parts:
- removed FB1: FerriteBead, symbol Device:FerriteBead
- added C14, C16: 12p, Capacitor_SMD:C_0402_1005Metric, symbol Device:C
- added C15, C17: 100n, Capacitor_SMD:C_0402_1005Metric, symbol Device:C
- added C18, C19, C20, C21, C22, C23, C24, C25, C26, C27, C28, C29: 22uF, Capacitor_SMD:C_Elec_6.3x7.7, symbol Device:C_Polarized
- added C2, C3: 10u, symbol Device:C
- added C30, C31, C32, C33, C34, C35, C36, C37, C38: 100n, Capacitor_SMD:C_0603_1608Metric, symbol Device:C
- added C39, C40, C41, C42, C43, C44, C45, C46, C47, C48: C, Capacitor_SMD:C_1210_3225Metric, symbol Device:C
- added C4: 100n, symbol Device:C
- added JP1: SolderJumper_2_Open, Jumper:SolderJumper-2_P1.3mm_Open_RoundedPad1.0x1.5mm, symbol Jumper:SolderJumper_2_Open
- added L1: 22u, symbol Device:L
- added NT1: NetTie_2, symbol Device:NetTie_2
- added R24: 1k, Resistor_SMD:R_0402_1005Metric, symbol Device:R
- added R25: 120, Resistor_SMD:R_1206_3216Metric, symbol Device:R
- added U2: TJA1044GTK/3, Package_SON:HVSON-8-1EP_3x3mm_P0.65mm_EP1.6x2.4mm, symbol User_Symbols:TJA1044GTK/3
- added Y1: 16MHz, Crystal:Crystal_SMD_3225-4Pin_3.2x2.5mm, symbol Device:Crystal_GND24
- C1: renamed from C4; value 100n -> 470n
- C5: value R -> 100n
- C6: value R -> 1u; footprint Capacitor_SMD:C_0402_1005Metric -> (none)
- C7: value R -> 220n; footprint Capacitor_SMD:C_0402_1005Metric -> (none)
- C8: value R -> 2u2; footprint Capacitor_SMD:C_0402_1005Metric -> (none)
- R1: renamed from R16; value R -> 33k
- R2: renamed from R17; value R -> 3k3
- renumbered NT4 to NT2, R24 to R3, R18 to R4, R19 to R5, R23 to R6, R20 to R7, R21 to R8
Connections:
- net +3V3: now also U1.1 (REG3/VDD), U1.2 (VBAT), C17.1, C2.1, C4.1, NT1.2, U2.5 (VIO); no longer C7.1, C8.1
- net +3V3A: now also NT1.1
- net GND: now also C14.1, C15.2, C16.1, C17.2, C2.2, C3.1, C4.2, U2.2 (GND), U2.9 (EPAD), Y1.2, Y1.4; no longer C7.2, C8.2
- net XTALI: now also C14.2, Y1.1
- net XTALO: now also R24.2
- net BFAST: now reaches C10.1, R7.2, R8.1
- net BSLOW: now reaches C9.1, R4.2, R5.1
- net CNRX: now reaches U1.47 (PA11)
- net CNRX: now also U2.4 (RXD)
- net CNTX: now reaches U1.48 (PA12)
- net CNTX: now also U2.1 (TXD)
- net +5V: now reaches U1.64 (REGIN)
- net +5V: now also C15.1, C3.2, U2.3 (VCC)
- net SWO: now reaches J1.6 (SWO)
- new net: JP1.2 (B), R25.2
- new net CANH: R25.1, U2.7 (CANH)
- new net CANL: JP1.1 (A), U2.6 (CANL)
- new net CNSTB: U2.8 (STB)
- new net XTALR: C16.2, R24.1, Y1.3
- no-connect marks 1 -> 0
Other:
- note added: "CAN"
- moved on the sheet: C10, C9, J1, NT2, R3, R4, R5, R6, R7, R8

Commit message: Save
Parts:
- added U3: 74HC595, Package_SO:SOIC-16_3.9x9.9mm_P1.27mm, symbol 74xx:74HC595
Changed lines of the file:
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@@
+	)
+	(symbol
+		(lib_id "74xx:74HC595")
+		(at 208.28 240.03 0)
+		(unit 1)
+		(exclude_from_sim no)
+		(in_bom yes)
+		(on_board yes)
+		(dnp no)
+		(fields_autoplaced yes)
+		(property "Reference" "U3"
+			(at 210.4233 222.25 0)
+			(effects
+				(font
+					(size 1.27 1.27)
+				)
+				(justify left)
+			)
+		)
+		(property "Value" "74HC595"
+			(at 210.4233 224.79 0)
+			(effects
+				(font
+					(size 1.27 1.27)
+				)
+				(justify left)
+			)
+		)
+		(property "Footprint" "Package_SO:SOIC-16_3.9x9.9mm_P1.27mm"
+			(at 208.28 240.03 0)
+			(effects
+				(font
+					(size 1.27 1.27)
+				)
+				(hide yes)
+			)
+		)
+		(property "Datasheet" "http://www.ti.com/lit/ds/symlink/sn74hc595.pdf"
+			(at 208.28 240.03 0)
+			(effects
+				(font
+					(size 1.27 1.27)
+				)
+				(hide yes)
+			)
+		)
+		(property "Description" "8-bit serial in/out Shift Register 3-State Outputs"
+			(at 208.28 240.03 0)
+			(effects
+				(font
+					(size 1.27 1.27)
+				)
+				(hide yes)
+			)
+		)
+		(property "LCSC" "C5947"
+			(at 208.28 240.03 0)
+			(effects
+				(font
+					(size 1.27 1.27)
+				)
+				(hide yes)
+			)
+		)
+		(pin "4"
+		)
+		(pin "7"
+		)
+		(pin "2"
+		)
+		(pin "5"
+		)
+		(pin "15"
+		)
+		(pin "8"
+		)
+		(pin "16"
+		)
+		(pin "13"
+		)
+		(pin "12"
+		)
+		(pin "10"
+		)
+		(pin "11"
+		)
+		(pin "9"
+		)
+		(pin "1"
+		)
+		(pin "14"
+		)
+		(pin "3"
+		)
+		(pin "6"
+		)
+		(instances
+			(project ""
+				(path "/38b0a34b-2047-47f6-90d7-ccdf77e8e212"
+					(reference "U3")
+					(unit 1)
+				)
+			)
+		)
 	)
 	(symbol
